File: IQ Tayloe Mixer.sch (KiCad schematic (older format))
At the start: 69 parts, among them J1 Audio_Jack, J2 PCB_SMA, J3 Pad, J4 Pad, J5 PCB_SMA, J6 PCB_SMA, T1 T50_SPLITTER, U1 LM358, U2 LM358, U3 LM358, U4 LM358, U5 LM358, U8 MCP1703A-2502_SOT223

Commit message: hh
Parts:
- C10, C11, C12, C13: symbol phase_v3-eagle-import:1.0UF-0805-25V-(+80_-20%) -> IQ-Tayloe-Mixer-rescue:1.0UF-0805-25V-(+80_-20%)-phase_v3-eagle-import
- C14: symbol Tayloe_Detector_v5-eagle-import:C5_3.5 -> IQ-Tayloe-Mixer-rescue:C5_3.5-Tayloe_Detector_v5-eagle-import
- R1, R10, R15, R16, R2, R5, R6, R9: symbol phase_v3-eagle-import:0.3OHM-0805-1_8W-1% -> IQ-Tayloe-Mixer-rescue:0.3OHM-0805-1_8W-1%-phase_v3-eagle-import
- U$1: symbol Tayloe_Detector_v5-eagle-import:FST3253 -> IQ-Tayloe-Mixer-rescue:FST3253-Tayloe_Detector_v5-eagle-import
Changed lines of the file:
@@
 	8800 8300 8800 7400
 $Comp
-L Tayloe_Detector_v5-eagle-import:GND #GND01
+L IQ-Tayloe-Mixer-rescue:GND-Tayloe_Detector_v5-eagle-import #GND01
 U 1 1 12C122FD
 P 9200 7200
@@
 $EndComp
 $Comp
-L Tayloe_Detector_v5-eagle-import:C5_3.5 C14
+L IQ-Tayloe-Mixer-rescue:C5_3.5-Tayloe_Detector_v5-eagle-import C14
 U 1 1 5EE9C731
 P 9900 6000
@@
 	5000 6400 5000 6000
 $Comp
-L phase_v3-eagle-import:0.3OHM-0805-1_8W-1% R1
+L IQ-Tayloe-Mixer-rescue:0.3OHM-0805-1_8W-1%-phase_v3-eagle-import R1
 U 1 1 5EF82F89
 P 2600 6000
@@
 $EndComp
 $Comp
-L phase_v3-eagle-import:0.3OHM-0805-1_8W-1% R5
+L IQ-Tayloe-Mixer-rescue:0.3OHM-0805-1_8W-1%-phase_v3-eagle-import R5
 U 1 1 5EF82F8F
 P 3000 6400
@@
 $EndComp
 $Comp
-L phase_v3-eagle-import:0.3OHM-0805-1_8W-1% R9
+L IQ-Tayloe-Mixer-rescue:0.3OHM-0805-1_8W-1%-phase_v3-eagle-import R9
 U 1 1 5EF82F95
 P 4800 6000
@@
 $EndComp
 $Comp
-L phase_v3-eagle-import:0.3OHM-0805-1_8W-1% R15
+L IQ-Tayloe-Mixer-rescue:0.3OHM-0805-1_8W-1%-phase_v3-eagle-import R15
 U 1 1 5EF82F9B
 P 5200 6400
@@
 $EndComp
 $Comp
-L phase_v3-eagle-import:0.3OHM-0805-1_8W-1% R2
+L IQ-Tayloe-Mixer-rescue:0.3OHM-0805-1_8W-1%-phase_v3-eagle-import R2
 U 1 1 5EF82FC5
 P 2600 7500
@@
 $EndComp
 $Comp
-L phase_v3-eagle-import:0.3OHM-0805-1_8W-1% R6
+L IQ-Tayloe-Mixer-rescue:0.3OHM-0805-1_8W-1%-phase_v3-eagle-import R6
 U 1 1 5EF82FCB
 P 3000 7900
@@
 $EndComp
 $Comp
-L phase_v3-eagle-import:0.3OHM-0805-1_8W-1% R10
+L IQ-Tayloe-Mixer-rescue:0.3OHM-0805-1_8W-1%-phase_v3-eagle-import R10
 U 1 1 5EF82FD1
 P 4800 7500
@@
 $EndComp
 $Comp
-L phase_v3-eagle-import:0.3OHM-0805-1_8W-1% R16
+L IQ-Tayloe-Mixer-rescue:0.3OHM-0805-1_8W-1%-phase_v3-eagle-import R16
 U 1 1 5EF82FD7
 P 5200 7900
@@
 	9200 6900 9200 7100
 $Comp
-L Tayloe_Detector_v5-eagle-import:FST3253 U$1
+L IQ-Tayloe-Mixer-rescue:FST3253-Tayloe_Detector_v5-eagle-import U$1
 U 1 1 6E1B97F5
 P 12000 7100
@@
 $EndComp
 $Comp
-L phase_v3-eagle-import:1.0UF-0805-25V-(+80_-20%) C10
+L IQ-Tayloe-Mixer-rescue:1.0UF-0805-25V-(+80_-20%)-phase_v3-eagle-import C10
 U 1 1 5EEBD3D7
 P 7550 6850
@@
 $EndComp
 $Comp
-L phase_v3-eagle-import:1.0UF-0805-25V-(+80_-20%) C11
+L IQ-Tayloe-Mixer-rescue:1.0UF-0805-25V-(+80_-20%)-phase_v3-eagle-import C11
 U 1 1 5EEBE874
 P 7550 7300
@@
 $EndComp
 $Comp
-L phase_v3-eagle-import:1.0UF-0805-25V-(+80_-20%) C12
+L IQ-Tayloe-Mixer-rescue:1.0UF-0805-25V-(+80_-20%)-phase_v3-eagle-import C12
 U 1 1 5EED34B4
 P 7550 7750
@@
 $EndComp
 $Comp
-L phase_v3-eagle-import:1.0UF-0805-25V-(+80_-20%) C13
+L IQ-Tayloe-Mixer-rescue:1.0UF-0805-25V-(+80_-20%)-phase_v3-eagle-import C13
 U 1 1 5EED8105
 P 7550 8200
